Commit message: Apply stashed changes and resolve README conflict

File: ROS/Quadruped/src/delto_m_ros2/dg_description/urdf/dg4f.urdf.xacro (robot description, xacro)
@@ -1,5 +1,5 @@
 <?xml version="1.0"?>
 <robot xmlns:xacro="http://wiki.ros.org/xacro">
-  <xacro:macro name="dg4f" params="prefix">
+  <xacro:macro name="dg4f" params="prefix use_gazebo">
     <material name="${prefix}silver">
       <color rgba="0.700 0.700 0.700 1.000"/>
@@ -815,4 +815,229 @@
       <child link="${prefix}l_dg_4_tip" />
     </joint>
+    <xacro:if value="${use_gazebo}">
+      <ros2_control name="${prefix}GripperGazeboSystem" type="system">
+        <hardware>
+            <plugin>gz_ros2_control/GazeboSimSystem</plugin>
+        </hardware>
+        <joint name="${prefix}j_dg_1_1">
+            <command_interface name="position">
+                <param name="min_position">-3.14</param>
+                <param name="max_position">3.14</param>
+            </command_interface>
+            <state_interface name="position">
+                <param name="initial_position">0.0</param>
+            </state_interface>
+            <state_interface name="velocity" />
+            <state_interface name="effort" />
+        </joint>
+        <joint name="${prefix}j_dg_1_2">
+            <command_interface name="position">
+                <param name="min_position">-3.14</param>
+                <param name="max_position">3.14</param>
+            </command_interface>
+            <state_interface name="position">
+                <param name="initial_position">1.5</param>
+            </state_interface>
+            <state_interface name="velocity" />
+            <state_interface name="effort" />
+        </joint>
+        <joint name="${prefix}j_dg_1_3">
+            <command_interface name="position">
+                <param name="min_position">-3.14</param>
+                <param name="max_position">3.14</param>
+            </command_interface>
+            <state_interface name="position">
+                <param name="initial_position">0.0</param>
+            </state_interface>
+            <state_interface name="velocity" />
+            <state_interface name="effort" />
+        </joint>
+        <joint name="${prefix}j_dg_1_4">
+            <command_interface name="position">
+                <param name="min_position">-3.14</param>
+                <param name="max_position">3.14</param>
+            </command_interface>
+            <state_interface name="position">
+                <param name="initial_position">0.0</param>
+            </state_interface>
+            <state_interface name="velocity" />
+            <state_interface name="effort" />
+        </joint>
+        <joint name="${prefix}j_dg_2_1">
+            <command_interface name="position">
+                <param name="min_position">-0.5</param>
+                <param name="max_position">0.5</param>
+            </command_interface>
+            <state_interface name="position">
+                <param name="initial_position">0.0</param>
+            </state_interface>
+            <state_interface name="velocity" />
+            <state_interface name="effort" />
+        </joint>
+        <joint name="${prefix}j_dg_2_2">
+            <command_interface name="position">
+                <param name="min_position">-0.5</param>
+                <param name="max_position">0.5</param>
+            </command_interface>
+            <state_interface name="position">
+                <param name="initial_position">1.5</param>
+            </state_interface>
+            <state_interface name="velocity" />
+            <state_interface name="effort" />
+        </joint>
+        <joint name="${prefix}j_dg_2_3">
+            <command_interface name="position">
+                <param name="min_position">-0.5</param>
+                <param name="max_position">0.5</param>
+            </command_interface>
+            <state_interface name="position">
+                <param name="initial_position">0.0</param>
+            </state_interface>
+            <state_interface name="velocity" />
+            <state_interface name="effort" />
+        </joint>
+        <joint name="${prefix}j_dg_2_4">
+            <command_interface name="position">
+                <param name="min_position">-0.5</param>
+                <param name="max_position">0.5</param>
+            </command_interface>
+            <state_interface name="position">
+                <param name="initial_position">0.0</param>
+            </state_interface>
+            <state_interface name="velocity" />
+            <state_interface name="effort" />
+        </joint>
+        <joint name="${prefix}j_dg_3_1">
+            <command_interface name="position">
+                <param name="min_position">-0.5</param>
+                <param name="max_position">0.5</param>
+            </command_interface>
+            <state_interface name="position">
+                <param name="initial_position">0.0</param>
+            </state_interface>
+            <state_interface name="velocity" />
+            <state_interface name="effort" />
+        </joint>
+        <joint name="${prefix}j_dg_3_2">
+            <command_interface name="position">
+                <param name="min_position">-0.5</param>
+                <param name="max_position">0.5</param>
+            </command_interface>
+            <state_interface name="position">
+                <param name="initial_position">1.5</param>
+            </state_interface>
+            <state_interface name="velocity" />
+            <state_interface name="effort" />
+        </joint>
+        <joint name="${prefix}j_dg_3_3">
+            <command_interface name="position">
+                <param name="min_position">-0.5</param>
+                <param name="max_position">0.5</param>
+            </command_interface>
+            <state_interface name="position">
+                <param name="initial_position">0.0</param>
+            </state_interface>
+            <state_interface name="velocity" />
+            <state_interface name="effort" />
+        </joint>
+        <joint name="${prefix}j_dg_3_4">
+            <command_interface name="position">
+                <param name="min_position">-0.5</param>
+                <param name="max_position">0.5</param>
+            </command_interface>
+            <state_interface name="position">
+                <param name="initial_position">0.0</param>
+            </state_interface>
+            <state_interface name="velocity" />
+            <state_interface name="effort" />
+        </joint>
+        <joint name = "${prefix}j_dg_4_1">
+            <command_interface name="position">
+                <param name="min_position">-0.5</param>
+                <param name="max_position">0.5</param>
+            </command_interface>
+            <state_interface name="position">
+                <param name="initial_position">0.0</param>
+            </state_interface>
+            <state_interface name="velocity" />
+            <state_interface name="effort" />
+        </joint>
+        <joint name = "${prefix}j_dg_4_2">
+            <command_interface name="position">
+                <param name="min_position">-0.5</param>
+                <param name="max_position">0.5</param>
+            </command_interface>
+            <state_interface name="position">
+                <param name="initial_position">1.5</param>
+            </state_interface>
+            <state_interface name="velocity" />
+            <state_interface name="effort" />
+        </joint>
+        <joint name = "${prefix}j_dg_4_3">
+            <command_interface name="position">
+                <param name="min_position">-0.5</param>
+                <param name="max_position">0.5</param>
+            </command_interface>
+            <state_interface name="position">
+                <param name="initial_position">0.0</param>
+            </state_interface>
+            <state_interface name="velocity" />
+            <state_interface name="effort" />
+        </joint>
+        <joint name = "${prefix}j_dg_4_4">
+            <command_interface name="position">
+                <param name="min_position">-0.5</param>
+                <param name="max_position">0.5</param>
+            </command_interface>
+            <state_interface name="position">
+                <param name="initial_position">0.0</param>
+            </state_interface>
+            <state_interface name="velocity" />
+            <state_interface name="effort" />
+        </joint>
+        <joint name = "${prefix}j_dg_1_inner">
+            <command_interface name="position">
+                <param name="min_position">-3.14</param>
+                <param name="max_position">3.14</param>
+            </command_interface>
+            <state_interface name="position">
+                <param name="initial_position">0.0</param>
+            </state_interface>
+            <state_interface name="velocity" />
+            <state_interface name="effort" />
+        </joint>
+        <joint name = "${prefix}j_dg_4_inner">
+            <command_interface name="position">
+                <param name="min_position">-3.14</param>
+                <param name="max_position">3.14</param>
+            </command_interface>
+            <state_interface name="position">
+                <param name="initial_position">0.0</param>
+            </state_interface>
+            <state_interface name="velocity" />
+            <state_interface name="effort" />
+        </joint>
+        <joint name="${prefix}j_dg_1_outer" mimic="true">
+            <state_interface name="position"/>
+            <state_interface name="velocity"/>
+            <state_interface name="effort"/>
+        </joint>
+        <joint name="${prefix}j_dg_1_mimic" mimic="true">
+            <state_interface name="position"/>
+            <state_interface name="velocity"/>
+            <state_interface name="effort"/>
+        </joint>
+        <joint name="${prefix}j_dg_4_outer" mimic="true">
+            <state_interface name="position"/>
+            <state_interface name="velocity"/>
+            <state_interface name="effort"/>
+        </joint>
+        <joint name="${prefix}j_dg_4_mimic" mimic="true">
+            <state_interface name="position"/>
+            <state_interface name="velocity"/>
+            <state_interface name="effort"/>
+        </joint>
+      </ros2_control>
+    </xacro:if>
   </xacro:macro>
 </robot>
