Commit message: Apply stashed changes and resolve README conflict

File: ROS/Quadruped/src/mm_description/urdf/obotx_dual_arm.urdf.xacro (robot description, xacro)
@@ -25,8 +25,6 @@
     <!-- ================= IMPORTS ================= -->
     <xacro:include filename="$(find summit_xl_description)/robots/summit_xls.urdf.xacro"/>
-    <xacro:include filename="$(find mm_description)/urdf/arm/arm.urdf.xacro"/>
-    <!-- <xacro:include filename="$(find mm_description)/urdf/base/mecanum_vehicle.urdf.xacro"/> -->
-    <!-- ================= 1. MOBILE BASE ================= -->
-    <!-- <xacro:mecanum_vehicle prefix="$(arg prefix)"/> -->
+    <xacro:include filename="$(find mm_description)/urdf/arm/morph1_arm.urdf.xacro"/>
+    <!-- ================= MOBILE BASE ================= -->
     <xacro:summit_xl prefix="$(arg prefix)" publish_bf="true" hq="$(arg hq)"/>
     <!-- ================= 2. LEFT ARM ================= -->
@@ -43,6 +41,6 @@
         <dynamics damping="0.1" friction="0.1"/>
     </joint>
-    <xacro:arm prefix="$(arg prefix)left_" use_gazebo="$(arg use_gazebo)"/>
-    <!-- ================= 3. RIGHT ARM ================= -->
+    <xacro:morph1_arm prefix="$(arg prefix)left_" use_gazebo="$(arg use_gazebo)"/>
+    <!-- ================= RIGHT ARM ================= -->
     <joint name="$(arg prefix)right_arm_mount_joint" type="revolute">
         <parent link="$(arg prefix)base_link_platform"/>
@@ -57,586 +55,37 @@
         <dynamics damping="0.1" friction="0.1"/>
     </joint>
-    <xacro:arm prefix="$(arg prefix)right_" use_gazebo="$(arg use_gazebo)"/>
-    <!-- ================= 4. MERGED ROS2_CONTROL ================= -->
+    <xacro:morph1_arm prefix="$(arg prefix)right_" use_gazebo="$(arg use_gazebo)"/>
+    <!-- ================= ROS2_CONTROL ================= -->
     <xacro:if value="$(arg use_gazebo)">
         <!-- Gazebo plugin -->
         <gazebo>
-        <plugin filename="gz_ros2_control-system"
-                name="gz_ros2_control::GazeboSimROS2ControlPlugin">
-            <parameters>$(find mm_control)/config/obotx_dual_arm_controllers.yaml</parameters>
-            <ros>
-                <remapping>/mecanum_drive_controller/reference:=/cmd_vel</remapping>
-                <remapping>/mecanum_drive_controller/odom:=/odom</remapping>
-            </ros>
-        </plugin>
+            <plugin filename="gz_ros2_control-system" name="gz_ros2_control::GazeboSimROS2ControlPlugin">
+                <parameters>$(find mm_control)/config/obotx_dual_arm_controllers.yaml</parameters>
+                <ros>
+                    <!-- <remapping>/mecanum_drive_controller/cmd_vel:=/cmd_vel</remapping> -->
+                    <remapping>/controller_manager/robot_description:=/robot_description</remapping>
+                </ros>
+            </plugin>
         </gazebo>
         <!-- Hardware definition -->
-        <ros2_control name="GazeboSystem" type="system">
-        <hardware>
-            <plugin>gz_ros2_control/GazeboSimSystem</plugin>
-        </hardware>
-        <!-- ===== MOBILE BASE WHEELS ===== -->
-        <joint name="$(arg prefix)front_left_wheel_joint">
-            <command_interface name="velocity">
-                <param name="min">-1</param>
-                <param name="max">1</param>
-            </command_interface>
-            <state_interface name="position"/>
-            <state_interface name="velocity"/>
-        </joint>
-        <joint name="$(arg prefix)front_right_wheel_joint">
-            <command_interface name="velocity">
-                <param name="min">-1</param>
-                <param name="max">1</param>
-            </command_interface>
-            <state_interface name="position"/>
-            <state_interface name="velocity"/>
-        </joint>
-        <joint name="$(arg prefix)rear_left_wheel_joint">
-            <command_interface name="velocity">
-                <param name="min">-1</param>
-                <param name="max">1</param>
-            </command_interface>
-            <state_interface name="position"/>
-            <state_interface name="velocity"/>
-        </joint>
-        <joint name="$(arg prefix)rear_right_wheel_joint">
-            <command_interface name="velocity">
-                <param name="min">-1</param>
-                <param name="max">1</param>
-            </command_interface>
-            <state_interface name="position"/>
-            <state_interface name="velocity"/>
-        </joint>
-        <joint name="$(arg prefix)left_joint_slider_right_hinge" mimic="true">
-            <state_interface name="position"/>
-            <state_interface name="velocity"/>
-            <state_interface name="effort"/>
-        </joint>
-        <!-- ===== LEFT ARM JOINTS ===== -->
-        <joint name="$(arg prefix)left_arm_mount_joint">
-            <command_interface name="position"/>
-            <state_interface name="position"/>
-            <state_interface name="velocity"/>
-            <state_interface name="effort"/>
-        </joint>
-        <joint name="$(arg prefix)left_joint_slider_left_slide">
-            <command_interface name="position"/>
-            <state_interface name="position"/>
-            <state_interface name="velocity"/>
-            <state_interface name="effort"/>
-        </joint>
-        <joint name="$(arg prefix)left_joint_slider_left_hinge">
-            <command_interface name="position"/>
-            <state_interface name="position"/>
-            <state_interface name="velocity"/>
-            <state_interface name="effort"/>
-        </joint>
-        <joint name="$(arg prefix)left_joint_telescopic_slide">
-            <command_interface name="position"/>
-            <state_interface name="position"/>
-            <state_interface name="velocity"/>
-            <state_interface name="effort"/>
-        </joint>
-        <joint name="$(arg prefix)left_joint_hinge_telescopic_hand">
-            <command_interface name="position"/>
-            <state_interface name="position"/>
-            <state_interface name="velocity"/>
-            <state_interface name="effort"/>
-        </joint>
-        <joint name="$(arg prefix)left_joint_slider_right_slide">
-            <command_interface name="position"/>
-            <state_interface name="position"/>
-            <state_interface name="velocity"/>
-            <state_interface name="effort"/>
-        </joint>
-        <!-- ===== RIGHT ARM JOINTS ===== -->
-        <joint name="$(arg prefix)right_arm_mount_joint">
-            <command_interface name="position"/>
-            <state_interface name="position"/>
-            <state_interface name="velocity"/>
-            <state_interface name="effort"/>
-        </joint>
-        <joint name="$(arg prefix)right_joint_slider_left_slide">
-            <command_interface name="position"/>
-            <state_interface name="position"/>
-            <state_interface name="velocity"/>
-            <state_interface name="effort"/>
-        </joint>
-        <joint name="$(arg prefix)right_joint_slider_left_hinge">
-            <command_interface name="position"/>
-            <state_interface name="position"/>
-            <state_interface name="velocity"/>
-            <state_interface name="effort"/>
-        </joint>
-        <joint name="$(arg prefix)right_joint_telescopic_slide">
-            <command_interface name="position"/>
-            <state_interface name="position"/>
-            <state_interface name="velocity"/>
-            <state_interface name="effort"/>
-        </joint>
-        <joint name="$(arg prefix)right_joint_hinge_telescopic_hand">
-            <command_interface name="position"/>
-            <state_interface name="position"/>
-            <state_interface name="velocity"/>
-            <state_interface name="effort"/>
-        </joint>
-        <joint name="$(arg prefix)right_joint_slider_right_slide">
-            <command_interface name="position"/>
-            <state_interface name="position"/>
-            <state_interface name="velocity"/>
-            <state_interface name="effort"/>
-        </joint>
-        <joint name="$(arg prefix)right_joint_slider_right_hinge" mimic="true">
-            <state_interface name="position"/>
-            <state_interface name="velocity"/>
-            <state_interface name="effort"/>
-            <state_interface name="effort"/>
-        </joint>
-        <!-- ===== DG4F GRIPPER JOINTS (Prefixed) ===== -->
-        <joint name="$(arg prefix)left_j_dg_1_1">
-            <command_interface name="position">
-                <param name="min_position">-3.14</param>
-                <param name="max_position">3.14</param>
-            </command_interface>
-            <state_interface name="position">
-                <param name="initial_position">0.0</param>
-            </state_interface>
-            <state_interface name="velocity" />
-            <state_interface name="effort" />
-        </joint>
-        <joint name="$(arg prefix)left_j_dg_1_2">
-            <command_interface name="position">
-                <param name="min_position">-3.14</param>
-                <param name="max_position">3.14</param>
-            </command_interface>
-            <state_interface name="position">
-                <param name="initial_position">1.5</param>
-            </state_interface>
-            <state_interface name="velocity" />
-            <state_interface name="effort" />
-        </joint>
-        <joint name="$(arg prefix)left_j_dg_1_3">
-            <command_interface name="position">
-                <param name="min_position">-3.14</param>
-                <param name="max_position">3.14</param>
-            </command_interface>
-            <state_interface name="position">
-                <param name="initial_position">0.0</param>
-            </state_interface>
-            <state_interface name="velocity" />
-            <state_interface name="effort" />
-        </joint>
-        <joint name="$(arg prefix)left_j_dg_1_4">
-            <command_interface name="position">
-                <param name="min_position">-3.14</param>
-                <param name="max_position">3.14</param>
-            </command_interface>
-            <state_interface name="position">
-                <param name="initial_position">0.0</param>
-            </state_interface>
-            <state_interface name="velocity" />
-            <state_interface name="effort" />
-        </joint>
-        <!-- Finger 2 joints -->
-        <joint name="$(arg prefix)left_j_dg_2_1">
-            <command_interface name="position">
-                <param name="min_position">-0.5</param>
-                <param name="max_position">0.5</param>
-            </command_interface>
-            <state_interface name="position">
-                <param name="initial_position">0.0</param>
-            </state_interface>
-            <state_interface name="velocity" />
-            <state_interface name="effort" />
-        </joint>
-        <joint name="$(arg prefix)left_j_dg_2_2">
-            <command_interface name="position">
-                <param name="min_position">-0.5</param>
-                <param name="max_position">0.5</param>
-            </command_interface>
-            <state_interface name="position">
-                <param name="initial_position">1.5</param>
-            </state_interface>
-            <state_interface name="velocity" />
-            <state_interface name="effort" />
-        </joint>
-        <joint name="$(arg prefix)left_j_dg_2_3">
-            <command_interface name="position">
-                <param name="min_position">-0.5</param>
-                <param name="max_position">0.5</param>
-            </command_interface>
-            <state_interface name="position">
-                <param name="initial_position">0.0</param>
-            </state_interface>
-            <state_interface name="velocity" />
-            <state_interface name="effort" />
-        </joint>
-        <joint name="$(arg prefix)left_j_dg_2_4">
-            <command_interface name="position">
-                <param name="min_position">-0.5</param>
-                <param name="max_position">0.5</param>
-            </command_interface>
-            <state_interface name="position">
-                <param name="initial_position">0.0</param>
-            </state_interface>
-            <state_interface name="velocity" />
-            <state_interface name="effort" />
-        </joint>
-        <!-- Finger 3 joints -->
-        <joint name="$(arg prefix)left_j_dg_3_1">
-            <command_interface name="position">
-                <param name="min_position">-0.5</param>
-                <param name="max_position">0.5</param>
-            </command_interface>
-            <state_interface name="position">
-                <param name="initial_position">0.0</param>
-            </state_interface>
-            <state_interface name="velocity" />
-            <state_interface name="effort" />
-        </joint>
-        <joint name="$(arg prefix)left_j_dg_3_2">
-            <command_interface name="position">
-                <param name="min_position">-0.5</param>
-                <param name="max_position">0.5</param>
-            </command_interface>
-            <state_interface name="position">
-                <param name="initial_position">1.5</param>
-            </state_interface>
-            <state_interface name="velocity" />
-            <state_interface name="effort" />
-        </joint>
-        <joint name="$(arg prefix)left_j_dg_3_3">
-            <command_interface name="position">
-                <param name="min_position">-0.5</param>
-                <param name="max_position">0.5</param>
-            </command_interface>
-            <state_interface name="position">
-                <param name="initial_position">0.0</param>
-            </state_interface>
-            <state_interface name="velocity" />
-            <state_interface name="effort" />
-        </joint>
-        <joint name="$(arg prefix)left_j_dg_3_4">
-            <command_interface name="position">
-                <param name="min_position">-0.5</param>
-                <param name="max_position">0.5</param>
-            </command_interface>
-            <state_interface name="position">
-                <param name="initial_position">0.0</param>
-            </state_interface>
-            <state_interface name="velocity" />
-            <state_interface name="effort" />
-        </joint>
-        <joint name = "$(arg prefix)left_j_dg_4_1">
-            <command_interface name="position">
-                <param name="min_position">-0.5</param>
-                <param name="max_position">0.5</param>
-            </command_interface>
-            <state_interface name="position">
-                <param name="initial_position">0.0</param>
-            </state_interface>
-            <state_interface name="velocity" />
-            <state_interface name="effort" />
-        </joint>
-        <joint name = "$(arg prefix)left_j_dg_4_2">
-            <command_interface name="position">
-                <param name="min_position">-0.5</param>
-                <param name="max_position">0.5</param>
-            </command_interface>
-            <state_interface name="position">
-                <param name="initial_position">1.5</param>
-            </state_interface>
-            <state_interface name="velocity" />
-            <state_interface name="effort" />
-        </joint>
-        <joint name = "$(arg prefix)left_j_dg_4_3">
-            <command_interface name="position">
-                <param name="min_position">-0.5</param>
-                <param name="max_position">0.5</param>
-            </command_interface>
-            <state_interface name="position">
-                <param name="initial_position">0.0</param>
-            </state_interface>
-            <state_interface name="velocity" />
-            <state_interface name="effort" />
-        </joint>
-        <joint name = "$(arg prefix)left_j_dg_4_4">
-            <command_interface name="position">
-                <param name="min_position">-0.5</param>
-                <param name="max_position">0.5</param>
-            </command_interface>
-            <state_interface name="position">
-                <param name="initial_position">0.0</param>
-            </state_interface>
-            <state_interface name="velocity" />
-            <state_interface name="effort" />
-        </joint>
-        <joint name = "$(arg prefix)left_j_dg_1_inner">
-            <command_interface name="position">
-                <param name="min_position">-3.14</param>
-                <param name="max_position">3.14</param>
-            </command_interface>
-            <state_interface name="position">
-                <param name="initial_position">0.0</param>
-            </state_interface>
-            <state_interface name="velocity" />
-            <state_interface name="effort" />
-        </joint>
-        <joint name = "$(arg prefix)left_j_dg_4_inner">
-            <command_interface name="position">
-                <param name="min_position">-3.14</param>
-                <param name="max_position">3.14</param>
-            </command_interface>
-            <state_interface name="position">
-                <param name="initial_position">0.0</param>
-            </state_interface>
-            <state_interface name="velocity" />
-            <state_interface name="effort" />
-        </joint>
-        <!-- MIMIC (Slave). NO command interface allowed. -->
-        <joint name="$(arg prefix)left_j_dg_1_outer" mimic="true">
-            <state_interface name="position"/>
-            <state_interface name="velocity"/>
-            <state_interface name="effort"/>
-        </joint>
-        <joint name="$(arg prefix)left_j_dg_1_mimic" mimic="true">
-            <state_interface name="position"/>
-            <state_interface name="velocity"/>
-            <state_interface name="effort"/>
-        </joint>
-        <joint name="$(arg prefix)left_j_dg_4_outer" mimic="true">
-            <state_interface name="position"/>
-            <state_interface name="velocity"/>
-            <state_interface name="effort"/>
-        </joint>
-        <joint name="$(arg prefix)left_j_dg_4_mimic" mimic="true">
-            <state_interface name="position"/>
-            <state_interface name="velocity"/>
-            <state_interface name="effort"/>
-        </joint>
-        <!-- ====================== RIGHT FINGERS =============== -->
-        <joint name="$(arg prefix)right_j_dg_1_1">
-            <command_interface name="position">
-                <param name="min_position">-3.14</param>
-                <param name="max_position">3.14</param>
-            </command_interface>
-            <state_interface name="position">
-                <param name="initial_position">0.0</param>
-            </state_interface>
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