Commit message: Apply stashed changes and resolve README conflict

File: ROS/Quadruped/src/summit_xl_common/summit_xl_description/robots/summit_xls.urdf.xacro (robot description, xacro)
@@ -9,5 +9,5 @@
 	<xacro:property name="wheel_offset_z" value="0.0" />
 	<xacro:property name="hq" value="true" />
-	<xacro:property name="roller_mu" value="1.5"/>
+	<xacro:property name="roller_mu" value="1.0"/>
 	<xacro:property name="roller_mu2" value="0.0"/>
 	<xacro:arg name="prefix" default="summit_xl_"/>
@@ -27,5 +27,4 @@
 			<origin xyz="-${wheel_offset_x} -${wheel_offset_y} ${wheel_offset_z}" rpy="0 0 0"/>
 		</xacro:omni_wheel>
-		<!-- Front-Left: ↘️ -45° roller axis -->
 		<gazebo reference="$(arg prefix)front_left_wheel">
 		<collision>
@@ -33,15 +32,15 @@
 			<friction>
 				<ode>
-				<mu>${roller_mu}</mu>
-				<mu2>${roller_mu2}</mu2>
-				<fdir1 gz:expressed_in="$(arg prefix)base_footprint_platform">1.0 -1.0 0.0</fdir1>
-				<kp>1000000.0</kp>
-        		<kd>1.0</kd>
+					<mu>${roller_mu}</mu>
+					<mu2>${roller_mu2}</mu2>
+					<!-- <fdir1 gz:expressed_in="$(arg prefix)base_footprint_platform">1.0 -1.0 0.0</fdir1> -->
 				</ode>
+				<torsional>
+					<coefficient>0.0</coefficient>
+				</torsional>
 			</friction>
 			</surface>
 		</collision>
 		</gazebo>
-		<!-- Rear-Left: ↗️ +45° roller axis -->
 		<gazebo reference="$(arg prefix)rear_left_wheel">
 		<collision>
@@ -49,15 +48,15 @@
 			<friction>
 				<ode>
-				<mu>${roller_mu}</mu>
-				<mu2>${roller_mu2}</mu2>
-				<fdir1 gz:expressed_in="$(arg prefix)base_footprint_platform">1.0 1.0 0.0</fdir1>
-				<kp>1000000.0</kp>
-        		<kd>1.0</kd>
+					<mu>${roller_mu}</mu>
+					<mu2>${roller_mu2}</mu2>
+					<!-- <fdir1 gz:expressed_in="$(arg prefix)base_footprint_platform">1.0 1.0 0.0</fdir1> -->
 				</ode>
+				<torsional>
+					<coefficient>0.0</coefficient>
+				</torsional>
 			</friction>
 			</surface>
 		</collision>
 		</gazebo>
-		<!-- Front-Right: ↗️ +45° roller axis -->
 		<gazebo reference="$(arg prefix)front_right_wheel">
 		<collision>
@@ -65,15 +64,15 @@
 			<friction>
 				<ode>
-				<mu>${roller_mu}</mu>
-				<mu2>${roller_mu2}</mu2>
-				<fdir1 gz:expressed_in="$(arg prefix)base_footprint_platform">1.0 1.0 0.0</fdir1>
-				<kp>1000000.0</kp>
-        		<kd>1.0</kd>
+					<mu>${roller_mu}</mu>
+					<mu2>${roller_mu2}</mu2>
+					<!-- <fdir1 gz:expressed_in="$(arg prefix)base_footprint_platform">1.0 1.0 0.0</fdir1> -->
 				</ode>
+				<torsional>
+					<coefficient>0.0</coefficient>
+				</torsional>
 			</friction>
 			</surface>
 		</collision>
 		</gazebo>
-		<!-- Rear-Right: ↘️ -45° roller axis -->
 		<gazebo reference="$(arg prefix)rear_right_wheel">
 		<collision>
@@ -81,18 +80,65 @@
 			<friction>
 				<ode>
-				<mu>${roller_mu}</mu>
-				<mu2>${roller_mu2}</mu2>
-				<fdir1 gz:expressed_in="$(arg prefix)base_footprint_platform">1.0 -1.0 0.0</fdir1>
-				<kp>1000000.0</kp>
-        		<kd>1.0</kd>
+					<mu>${roller_mu}</mu>
+					<mu2>${roller_mu2}</mu2>
+					<!-- <fdir1 gz:expressed_in="$(arg prefix)base_footprint_platform">1.0 -1.0 0.0</fdir1> -->
 				</ode>
+				<torsional>
+					<coefficient>0.0</coefficient>
+				</torsional>
 			</friction>
 			</surface>
 		</collision>
 		</gazebo>
-		<gazebo reference="$(arg prefix)base_link_platform">
+		<!-- <gazebo reference="$(arg prefix)base_link_platform">
 			<mu1>0.000002</mu1>
 			<mu2>0.000002</mu2>
-		</gazebo>
+		</gazebo> -->
+		<ros2_control name="${prefix}SummitXlGazeboSystem" type="system">
+			<hardware>
+				<plugin>gz_ros2_control/GazeboSimSystem</plugin>
+			</hardware>
+			<joint name="$(arg prefix)front_left_wheel_joint">
+				<command_interface name="velocity">
+					<param name="min">-50.0</param>
+					<param name="max">50.0</param>
+				</command_interface>
+				<state_interface name="position"/>
+				<state_interface name="velocity"/>
+			</joint>
+			<joint name="$(arg prefix)front_right_wheel_joint">
+				<command_interface name="velocity">
+					<param name="min">-50.0</param>
+					<param name="max">50.0</param>
+				</command_interface>
+				<state_interface name="position"/>
+				<state_interface name="velocity"/>
+			</joint>
+			<joint name="$(arg prefix)rear_left_wheel_joint">
+				<command_interface name="velocity">
+					<param name="min">-50.0</param>
+					<param name="max">50.0</param>
+				</command_interface>
+				<state_interface name="position"/>
+				<state_interface name="velocity"/>
+			</joint>
+			<joint name="$(arg prefix)rear_right_wheel_joint">
+				<command_interface name="velocity">
+					<param name="min">-50.0</param>
+					<param name="max">50.0</param>
+				</command_interface>
+				<state_interface name="position"/>
+				<state_interface name="velocity"/>
+			</joint>
+		</ros2_control>
+        <gazebo>
+            <plugin
+                filename="gz-sim-velocity-control-system"
+                name="gz::sim::systems::VelocityControl">
+                <topic>mecanum_drive_controller/cmd_vel</topic>
+                <initial_linear>0 0 0</initial_linear>
+                <initial_angular>0 0 0</initial_angular>
+            </plugin>
+        </gazebo>
    </xacro:macro>
 </robot>

File: ROS/Quadruped/src/summit_xl_common/summit_xl_description/urdf/wheels/basic_wheel.urdf.xacro (robot description, xacro)
@@ -26,5 +26,4 @@
           <cylinder length="${height}" radius="${radius}" />
         </geometry>
-        <material name="dark-gray"/>
       </visual>
       <collision>

File: ROS/Quadruped/src/summit_xl_common/summit_xl_description/urdf/wheels/omni_wheel.urdf.xacro (robot description, xacro)
@@ -17,6 +17,4 @@
       <xacro:insert_block name="origin" />
       <axis xyz="0 1 0" rpy="0 0 0" />
-      <limit effort="100000" velocity="100000"/>
-      <joint_properties damping="1.0" friction="1.0"/>
     </joint>
     <link name="${prefix}_wheel">
@@ -41,7 +39,4 @@
           </geometry>
         </xacro:unless>
-        <material name="darkgrey">
-           <color rgba="0.2 0.2 0.2 1"/>
-        </material>
       </visual>
       <collision>
@@ -49,15 +44,14 @@
         <geometry>
           <!--sphere radius="${omni_wheel_radius}" /-->
-<!--
-          <xacro:if value="${reflect}">
-              <mesh filename="file://$(find summit_xl_description)/meshes/wheels/omni_wheel_1.dae" />
-          </xacro:if>
-          <xacro:unless value="${reflect}">
-              <mesh filename="file://$(find summit_xl_description)/meshes/wheels/omni_wheel_2.dae" />
-					</xacro:unless>
--->
 					<cylinder length="${omni_wheel_height}" radius="${omni_wheel_radius}" />
 					<!-- sphere radius="${omni_wheel_radius}"/-->
         </geometry>
+        <surface>
+          <friction>
+            <torsional>
+              <coefficient>0.0</coefficient>
+            </torsional>
+          </friction>
+        </surface>
       </collision>
       <inertial>
