Commit message: feat: update descale gripper and add rqt joint control

File: ROS/Quadruped/src/mm_description/urdf/arm/morph1_arm.urdf.xacro (robot description, xacro)
@@ -5,11 +5,11 @@
     <xacro:property name="vertical_mesh_prefix" value="file://$(find mm_description)/meshes/arm/vertical_arm/morph_1"/>
     <xacro:property name="telescopic_mesh_prefix" value="file://$(find mm_description)/meshes/arm/telescopic_arm/morph_1"/>
-    <xacro:include filename="$(find mm_description)/urdf/gripper/robotiq_3f.urdf.xacro" />
+    <xacro:include filename="$(find mm_description)/urdf/gripper/robotiq_3f/robotiq_3f.urdf.xacro" />
     <xacro:robotiq_3f prefix="${prefix}" use_gazebo="${use_gazebo}"/>
-    <xacro:property name="slide_limit_min" value="-1"/>
-    <xacro:property name="slide_limit_max" value="1.112"/>
+    <xacro:property name="slide_limit_min" value="0"/>
+    <xacro:property name="slide_limit_max" value="1.312"/>
     <xacro:property name="hinge_limit_min" value="-3.14159"/>
     <xacro:property name="hinge_limit_max" value="3.14159"/>
-    <xacro:property name="telescopic_limit_min" value="-1"/>
+    <xacro:property name="telescopic_limit_min" value="0"/>
     <xacro:property name="telescopic_limit_max" value="0.5"/>
     <xacro:property name="telescopic_hinge_limit_min" value="-1.1345"/>
@@ -106,6 +106,6 @@
       <parent link="${prefix}hinge_telescopic_hand"/>
       <child link="${prefix}palm_wrist_roll"/>
-      <origin xyz="-0.107377 0 0" rpy="0 0 0"/>
-      <axis xyz="1 0 0"/>
+      <origin xyz="-0.08 0 0" rpy="0 0 0"/>
+      <axis xyz="0 0 1"/>
       <limit lower="${gripper_roll_limit_min}" upper="${gripper_roll_limit_max}"
             effort="${default_effort}" velocity="${default_velocity}"/>
@@ -127,5 +127,5 @@
       <child link="${prefix}base_link_palm"/>
       <origin xyz="0 0 0" rpy="0 0 0"/>
-      <axis xyz="0 0 1"/>
+      <axis xyz="1 0 0"/>
       <limit lower="${gripper_yaw_limit_min}" upper="${gripper_yaw_limit_max}"
             effort="${default_effort}" velocity="${default_velocity}"/>

File: ROS/Quadruped/src/mm_description/urdf/obotx_dual_arm.urdf.xacro (robot description, xacro)
@@ -12,6 +12,6 @@
     <xacro:arg name="left_arm_mount_p" default="0.0"/>
     <xacro:arg name="left_arm_mount_yaw" default="3.14159"/>
-    <xacro:arg name="arm_base_yaw_limit_lower" default="-3.14"/>
-    <xacro:arg name="arm_base_yaw_limit_upper" default="3.14"/>
+    <xacro:arg name="arm_base_yaw_limit_lower" default="-3.14159"/>
+    <xacro:arg name="arm_base_yaw_limit_upper" default="3.14159"/>
     <xacro:arg name="arm_base_yaw_effort" default="50"/>
     <xacro:arg name="arm_base_yaw_velocity" default="50.0"/>
@@ -24,8 +24,8 @@
     <xacro:arg name="right_arm_mount_yaw" default="3.14159"/>
     <!-- ================= IMPORTS ================= -->
-    <xacro:include filename="$(find summit_xl_description)/robots/summit_xls.urdf.xacro"/>
+    <xacro:include filename="$(find mm_description)/urdf/platform/summit_xl/summit_xls.urdf.xacro"/>
     <xacro:include filename="$(find mm_description)/urdf/arm/morph1_arm.urdf.xacro"/>
     <!-- ================= MOBILE BASE ================= -->
-    <xacro:summit_xl prefix="$(arg prefix)" publish_bf="true" hq="$(arg hq)"/>
+    <xacro:summit_xl prefix="$(arg prefix)"/>
     <!-- ================= 2. LEFT ARM ================= -->
     <joint name="$(arg prefix)left_arm_mount_joint" type="revolute">
@@ -61,5 +61,5 @@
         <gazebo>
             <plugin filename="gz_ros2_control-system" name="gz_ros2_control::GazeboSimROS2ControlPlugin">
-                <parameters>$(find mm_control)/config/obotx_dual_arm_controllers.yaml</parameters>
+                <parameters>$(find mm_control)/config/controller_manager/obotx_dual_arm_controllers.yaml</parameters>
                 <ros>
                     <!-- <remapping>/mecanum_drive_controller/cmd_vel:=/cmd_vel</remapping> -->
