Commit message: feat: moveit integraton

File: ROS/Quadruped/src/mm_description/urdf/gripper/robotiq_3f/robotiq_3f.urdf.xacro (robot description, xacro)
@@ -2,12 +2,10 @@
 <robot xmlns:xacro="http://ros.org/wiki/xacro" name="robotiq_3f_gripper">
   <xacro:macro name="robotiq_3f" params="prefix use_gazebo">
-    <!-- Mesh path property + scale factor -->
     <xacro:property name="gripper_mesh_prefix" value="file://$(find mm_description)/meshes/gripper/robotiq_3f"/>
     <xacro:property name="scale_factor" value="0.7"/>
-    <!-- Include scaled finger macro (ensure robotiq_3f_finger.xacro also has scale_factor defined) -->
     <xacro:include filename="$(find mm_description)/urdf/gripper/robotiq_3f/robotiq_3f_finger.xacro" />
-    <xacro:robotiq_3f_finger prefix="${prefix}finger_1_" scale_factor="${scale_factor}"/>
-    <xacro:robotiq_3f_finger prefix="${prefix}finger_2_" scale_factor="${scale_factor}"/>
-    <xacro:robotiq_3f_finger prefix="${prefix}finger_middle_" scale_factor="${scale_factor}"/>
+    <xacro:robotiq_3f_finger prefix="${prefix}finger_1_" scale_factor="${scale_factor}" use_gazebo="${use_gazebo}"/>
+    <xacro:robotiq_3f_finger prefix="${prefix}finger_2_" scale_factor="${scale_factor}" use_gazebo="${use_gazebo}"/>
+    <xacro:robotiq_3f_finger prefix="${prefix}finger_middle_" scale_factor="${scale_factor}" use_gazebo="${use_gazebo}"/>
     <!-- link list -->
     <link name="${prefix}base_link_palm"/>

File: ROS/Quadruped/src/mm_description/urdf/gripper/robotiq_3f/robotiq_3f_finger.xacro (robot description, xacro)
@@ -1,4 +1,4 @@
 <robot xmlns:xacro="http://ros.org/wiki/xacro">
-    <xacro:macro name="robotiq_3f_finger" params="prefix scale_factor">
+    <xacro:macro name="robotiq_3f_finger" params="prefix scale_factor use_gazebo">
 		<!-- Mesh path property -->
 		<xacro:property name="gripper_mesh_prefix" value="file://$(find mm_description)/meshes/gripper/robotiq_3f"/>
@@ -106,29 +106,32 @@
 		</joint>
 		<!-- end of joint list -->
-        <ros2_control name="${prefix}GripperFingerGazeboSystem" type="system">
-            <hardware>
-                <plugin>gz_ros2_control/GazeboSimSystem</plugin>
-            </hardware>
-            <joint name="${prefix}joint_1">
-                <command_interface name="position">
-                    <limits enable="false"/>
-                </command_interface>
-                <state_interface name="position"/>
-                <state_interface name="velocity"/>
-                <state_interface name="effort"/>
-            </joint>
-            <joint name="${prefix}joint_2">
-                <command_interface name="position"/>
-                <state_interface name="position"/>
-                <state_interface name="velocity"/>
-                <state_interface name="effort"/>
-            </joint>
-            <joint name="${prefix}joint_3">
-                <command_interface name="position"/>
-                <state_interface name="position"/>
-                <state_interface name="velocity"/>
-                <state_interface name="effort"/>
-            </joint>
-        </ros2_control>
+    	<xacro:if value="${use_gazebo}">
+			<ros2_control name="${prefix}GripperFingerGazeboSystem" type="system">
+				<hardware>
+					<plugin>gz_ros2_control/GazeboSimSystem</plugin>
+				</hardware>
+				<joint name="${prefix}joint_1">
+					<command_interface name="position"/>
+					<state_interface name="position">
+					</state_interface>
+					<state_interface name="velocity"/>
+					<state_interface name="effort"/>
+				</joint>
+				<joint name="${prefix}joint_2">
+					<command_interface name="position"/>
+					<state_interface name="position">
+					</state_interface>
+					<state_interface name="velocity"/>
+					<state_interface name="effort"/>
+				</joint>
+				<joint name="${prefix}joint_3">
+					<command_interface name="position"/>
+					<state_interface name="position">
+					</state_interface>
+					<state_interface name="velocity"/>
+					<state_interface name="effort"/>
+				</joint>
+			</ros2_control>
+		</xacro:if>
 	</xacro:macro>
 </robot>

File: ROS/Quadruped/src/mm_description/urdf/platform/summit_xl/omni_wheel.urdf.xacro (robot description, xacro)
@@ -17,9 +17,8 @@
       <xacro:insert_block name="origin" />
       <axis xyz="0 1 0" rpy="0 0 0" />
-      <limit effort="100" velocity="100.0" lower="-${M_PI}" upper="${M_PI}"/>
+      <limit effort="100000" velocity="100.0" lower="-${M_PI}" upper="${M_PI}"/>
     </joint>
     <link name="${prefix}_wheel">
       <visual>
-        <xacro:if value="${hq}">
           <origin xyz="0 0 0" rpy="0 0 0" />
           <xacro:if value="${reflect}">
@@ -32,12 +31,5 @@
               <mesh filename="file://$(find mm_description)/meshes/platform/summit_xl/omni_wheel_2.dae" />
             </geometry>
-		  </xacro:unless>
-        </xacro:if>
-        <xacro:unless value="${hq}">
-          <origin xyz="0 0 0" rpy="0 0 0" />
-          <geometry>
-            <sphere radius="${omni_wheel_radius}" />
-          </geometry>
-        </xacro:unless>
+		      </xacro:unless>
       </visual>
       <collision>

File: ROS/Quadruped/src/mm_description/urdf/platform/summit_xl/summit_xls.urdf.xacro (robot description, xacro)
@@ -8,9 +8,9 @@
 	<xacro:property name="wheel_offset_y" value="0.2045" />
 	<xacro:property name="wheel_offset_z" value="0.0" />
-	<xacro:property name="hq" value="true" />
-	<xacro:property name="roller_mu" value="1.0"/>
-	<xacro:property name="roller_mu2" value="0.0"/>
+	<xacro:property name="roller_mu" value="2.0"/>
+	<xacro:property name="roller_mu2" value="0.1"/>
 	<xacro:arg name="prefix" default="summit_xl_"/>
-    <xacro:macro name="summit_xl" params="prefix">
+	<xacro:arg name="use_gazebo" default="true"/>
+    <xacro:macro name="summit_xl" params="prefix use_gazebo">
 		<!-- Summit XL base -->
 		<xacro:summit_xls_base prefix="$(arg prefix)" />
@@ -34,5 +34,5 @@
 					<mu>${roller_mu}</mu>
 					<mu2>${roller_mu2}</mu2>
-					<!-- <fdir1 gz:expressed_in="$(arg prefix)base_footprint_platform">1.0 -1.0 0.0</fdir1> -->
+					<fdir1 gz:expressed_in="$(arg prefix)base_footprint_platform">1.0 -1.0 0.0</fdir1>
 				</ode>
 				<torsional>
@@ -50,5 +50,5 @@
 					<mu>${roller_mu}</mu>
 					<mu2>${roller_mu2}</mu2>
-					<!-- <fdir1 gz:expressed_in="$(arg prefix)base_footprint_platform">1.0 1.0 0.0</fdir1> -->
+					<fdir1 gz:expressed_in="$(arg prefix)base_footprint_platform">1.0 1.0 0.0</fdir1>
 				</ode>
 				<torsional>
@@ -66,5 +66,5 @@
 					<mu>${roller_mu}</mu>
 					<mu2>${roller_mu2}</mu2>
-					<!-- <fdir1 gz:expressed_in="$(arg prefix)base_footprint_platform">1.0 1.0 0.0</fdir1> -->
+					<fdir1 gz:expressed_in="$(arg prefix)base_footprint_platform">1.0 1.0 0.0</fdir1>
 				</ode>
 				<torsional>
@@ -82,5 +82,5 @@
 					<mu>${roller_mu}</mu>
 					<mu2>${roller_mu2}</mu2>
-					<!-- <fdir1 gz:expressed_in="$(arg prefix)base_footprint_platform">1.0 -1.0 0.0</fdir1> -->
+					<fdir1 gz:expressed_in="$(arg prefix)base_footprint_platform">1.0 -1.0 0.0</fdir1>
 				</ode>
 				<torsional>
@@ -95,50 +95,52 @@
 			<mu2>0.000002</mu2>
 		</gazebo> -->
-		<ros2_control name="${prefix}SummitXlGazeboSystem" type="system">
-			<hardware>
-				<plugin>gz_ros2_control/GazeboSimSystem</plugin>
-			</hardware>
-			<joint name="$(arg prefix)front_left_wheel_joint">
-				<command_interface name="velocity">
-					<param name="min">-50.0</param>
-					<param name="max">50.0</param>
-				</command_interface>
-				<state_interface name="position"/>
-				<state_interface name="velocity"/>
-			</joint>
-			<joint name="$(arg prefix)front_right_wheel_joint">
-				<command_interface name="velocity">
-					<param name="min">-50.0</param>
-					<param name="max">50.0</param>
-				</command_interface>
-				<state_interface name="position"/>
-				<state_interface name="velocity"/>
-			</joint>
-			<joint name="$(arg prefix)rear_left_wheel_joint">
-				<command_interface name="velocity">
-					<param name="min">-50.0</param>
-					<param name="max">50.0</param>
-				</command_interface>
-				<state_interface name="position"/>
-				<state_interface name="velocity"/>
-			</joint>
-			<joint name="$(arg prefix)rear_right_wheel_joint">
-				<command_interface name="velocity">
-					<param name="min">-50.0</param>
-					<param name="max">50.0</param>
-				</command_interface>
-				<state_interface name="position"/>
-				<state_interface name="velocity"/>
-			</joint>
-		</ros2_control>
-        <gazebo>
-            <plugin
-                filename="gz-sim-velocity-control-system"
-                name="gz::sim::systems::VelocityControl">
-                <topic>mecanum_drive_controller/cmd_vel</topic>
-                <initial_linear>0 0 0</initial_linear>
-                <initial_angular>0 0 0</initial_angular>
-            </plugin>
-        </gazebo>
+   		<xacro:if value="${use_gazebo}">
+			<ros2_control name="${prefix}SummitXlGazeboSystem" type="system">
+				<hardware>
+					<plugin>gz_ros2_control/GazeboSimSystem</plugin>
+				</hardware>
+				<joint name="$(arg prefix)front_left_wheel_joint">
+					<command_interface name="velocity">
+						<param name="min">-50.0</param>
+						<param name="max">50.0</param>
+					</command_interface>
+					<state_interface name="position"/>
+					<state_interface name="velocity"/>
+				</joint>
+				<joint name="$(arg prefix)front_right_wheel_joint">
+					<command_interface name="velocity">
+						<param name="min">-50.0</param>
+						<param name="max">50.0</param>
+					</command_interface>
+					<state_interface name="position"/>
+					<state_interface name="velocity"/>
+				</joint>
+				<joint name="$(arg prefix)rear_left_wheel_joint">
+					<command_interface name="velocity">
+						<param name="min">-50.0</param>
+						<param name="max">50.0</param>
+					</command_interface>
+					<state_interface name="position"/>
+					<state_interface name="velocity"/>
+				</joint>
+				<joint name="$(arg prefix)rear_right_wheel_joint">
+					<command_interface name="velocity">
+						<param name="min">-50.0</param>
+						<param name="max">50.0</param>
+					</command_interface>
+					<state_interface name="position"/>
+					<state_interface name="velocity"/>
+				</joint>
+			</ros2_control>
+			<gazebo>
+				<plugin
+					filename="gz-sim-velocity-control-system"
+					name="gz::sim::systems::VelocityControl">
+					<topic>mecanum_drive_controller/cmd_vel</topic>
+					<initial_linear>0 0 0</initial_linear>
+					<initial_angular>0 0 0</initial_angular>
+				</plugin>
+			</gazebo>
+		</xacro:if>
    </xacro:macro>
 </robot>

Commit message: feat: add moveit + nav2 pick and place, and delete 'mecanum_drive_controller' directly use mecanum control from ros2 controller

File: ROS/Quadruped/src/mm_description/urdf/gripper/robotiq_3f/robotiq_3f.urdf.xacro (robot description, xacro)
@@ -57,5 +57,5 @@
       <parent link="${prefix}palm"/>
       <child link="${prefix}tool0"/>
-      <origin xyz="0.0 ${0.1 * scale_factor} 0.0" rpy="0 0 1.5707"/>
+      <origin xyz="0.0 ${0.15 * scale_factor} 0.0" rpy="0 0 1.5707"/>
     </joint>
     <!-- end of joint list -->

File: ROS/Quadruped/src/mm_description/urdf/platform/summit_xl/summit_xls.urdf.xacro (robot description, xacro)
@@ -8,6 +8,6 @@
 	<xacro:property name="wheel_offset_y" value="0.2045" />
 	<xacro:property name="wheel_offset_z" value="0.0" />
-	<xacro:property name="roller_mu" value="2.0"/>
-	<xacro:property name="roller_mu2" value="0.1"/>
+	<xacro:property name="roller_mu" value="1.0"/>
+	<xacro:property name="roller_mu2" value="0.0"/>
 	<xacro:arg name="prefix" default="summit_xl_"/>
 	<xacro:arg name="use_gazebo" default="true"/>
@@ -133,5 +133,5 @@
 				</joint>
 			</ros2_control>
-			<gazebo>
+			<!-- <gazebo>
 				<plugin
 					filename="gz-sim-velocity-control-system"
@@ -141,5 +141,5 @@
 					<initial_angular>0 0 0</initial_angular>
 				</plugin>
-			</gazebo>
+			</gazebo> -->
 		</xacro:if>
    </xacro:macro>

File: ROS/Quadruped/src/mm_description/urdf/robot/morph_i.urdf.xacro (robot description, xacro)
@@ -63,5 +63,6 @@
                 <parameters>$(find mm_moveit_config)/config/morph_i/ros2_controllers.yaml</parameters>
                 <ros>
-                    <!-- <remapping>/mecanum_drive_controller/cmd_vel:=/cmd_vel</remapping> -->
+                    <remapping>/mecanum_drive_controller/reference:=/cmd_vel</remapping>
+                    <remapping>/mecanum_drive_controller/odometry:=/odom</remapping>
                     <remapping>/controller_manager/robot_description:=/robot_description</remapping>
                 </ros>
